Commit message: XML format and links repaired

File: src/bot_description/urdf/bot.urdf.xacro (robot description, xacro)
@@ -1,4 +1,4 @@
 <?xml version="1.0"?>
-<robot xlmns="http://www.ros.org/wiki/xacro" name="bot">
+<robot xmlns="http://www.ros.org/wiki/xacro" name="bot">
     <link name="base_footprint"/>
     <link name="base_link">
@@ -12,5 +12,5 @@
     <joint name="base joint" type="fixed">
         <parent link="base_footprint"/>
-        <child link="base_footprint"/>
+        <child link="base_link"/>
         <origin rpy="0 0 0" xyz="0 0 0.033"/>
     </joint>
