Commit message: plugin update

File: src/bot_description/urdf/bot_control.xacro (robot description, xacro)
@@ -12,4 +12,11 @@
             </hardware>
         </xacro:unless>
+        <joint name="wheel_right_joint">
+            <command_interface name="velocity">
+                <param name="min">-1</param>
+                <param name="max">1</param>
+            </command_interface>
+            <state_interface name="velocity"/>
+        </joint>
     </ros2_control>
 </robot>

File: src/bot_description/urdf/bot_gazebo.xacro (robot description, xacro)
@@ -35,3 +35,5 @@
         <maxVel>0.1</maxVel>
     </gazebo>
+    <gazebo>
+    </gazebo>
 </robot>
